File: PCB/RoboCon2025_PCB/RoboCon2025_ADIF-BB/RoboCon2025_ADIF-BB.kicad_sch (KiCad schematic)
At the start: 27 parts, among them J1 Conn_01x05, J2 Conn_01x09, J3 Conn_01x09, J4 S2B-XH-A, J6 S3B-XH-A, J7 S2B-XH-A, J8 S2B-XH-A, J9 S3B-XH-A, U1 PCM5102A, U3 TBD62083AFNG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

Commit message: [PCB] update: BB基板のパターン引いた(未配線あり)
Parts:
- D1, D2: footprint Diode_THT:D_DO-15_P2.54mm_Vertical_AnodeUp -> Diode_THT:D_A-405_P7.62mm_Horizontal
- R7, R8, R9: footprint Resistor_THT:R_Axial_DIN0207_L6.3mm_D2.5mm_P2.54mm_Vertical -> Resistor_THT:R_Axial_DIN0204_L3.6mm_D1.6mm_P7.62mm_Horizontal
Connections:
- net ACT_N: now also U4.23 (GPA2); no longer U4.27 (GPA6)
- net AUDIO_OUT_L: now also J6.3 (Pin_3); no longer J6.2 (Pin_2)
- net AUDIO_OUT_R: now also J6.2 (Pin_2); no longer J6.3 (Pin_3)
- net EXT_3SDA: no longer J2.7 (Pin_7)
- net GND: no longer J3.5 (Pin_5)
- net at U3.5 (I5): now also U4.24 (GPA3); no longer U4.26 (GPA5)
- net at U3.7 (I7): now also U4.27 (GPA6); no longer U4.24 (GPA3)
- net at U3.8 (I8): now also U4.26 (GPA5); no longer U4.23 (GPA2)
- no-connect marks 29 -> 31
Other:
- moved on the sheet: J6, R9

Commit message: [PCB] update: 配線完了！
Connections:
- net ACT_N: now also U4.24 (GPA3); no longer U4.23 (GPA2)
- net AUDIO_OUT_L: now also J6.2 (Pin_2); no longer J6.3 (Pin_3)
- net AUDIO_OUT_R: now also J6.3 (Pin_3); no longer J6.2 (Pin_2)
- net GND: now also J3.9 (Pin_9), U4.7 (GPB6); no longer J2.9 (Pin_9)
- net at U3.5 (I5): now also U4.25 (GPA4); no longer U4.24 (GPA3)
- net at U3.6 (I6): now also U4.26 (GPA5); no longer U4.25 (GPA4)
- net at U3.7 (I7): now also U4.28 (GPA7); no longer U4.27 (GPA6)
- net at U3.8 (I8): now also U4.27 (GPA6); no longer U4.26 (GPA5)
- no-connect marks 31 -> 30
Other:
- moved on the sheet: J6, R9
