File: PCB/RoboCon2025_PCB/RoboCon2025_ADIF-BB-P/RoboCon2025_ADIF-BB-P.kicad_pcb (KiCad board)
At the start: 2 copper layers, 47 x 72 mm, 12 parts, among them J1 Conn_01x05, J2 Conn_01x09, J3 Conn_01x09, J4 S2B-XH-A, J5 S3B-XH-A, U1 MCP23017_SP, U2 TBD62083AFNG

Commit message: [PCB] update: 配線完了！
Changed lines of the file:
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@@
 		(start 127 66.04)
 		(end 124.46 66.04)
-		(width 0.2)
+		(width 0.8)
 		(layer "F.Cu")
 		(net 1)
@@
 		(start 160.02 60.96)
 		(end 160.02 71.12)
-		(width 0.2)
+		(width 0.8)
 		(layer "B.Cu")
 		(net 1)
@@
 		(start 129.54 71.12)
 		(end 132.08 71.12)
-		(width 0.2)
+		(width 0.8)
 		(layer "B.Cu")
 		(net 1)
@@
 		(start 142.24 88.9)
 		(end 137.16 88.9)
-		(width 0.2)
+		(width 0.8)
 		(layer "B.Cu")
 		(net 1)
@@
 		(start 160.02 58.42)
 		(end 160.02 60.96)
-		(width 0.2)
+		(width 0.8)
 		(layer "B.Cu")
 		(net 1)
@@
 		(start 157.48 88.9)
 		(end 157.48 71.12)
-		(width 0.2)
+		(width 0.8)
 		(layer "B.Cu")
 		(net 1)
@@
 		(start 129.54 66.04)
 		(end 127 66.04)
-		(width 0.2)
+		(width 0.8)
 		(layer "B.Cu")
 		(net 1)
@@
 		(start 160.02 71.12)
 		(end 157.48 71.12)
-		(width 0.2)
+		(width 0.8)
 		(layer "B.Cu")
 		(net 1)
@@
 		(start 137.16 88.9)
 		(end 132.08 88.9)
-		(width 0.2)
+		(width 0.8)
 		(layer "B.Cu")
 		(net 1)
@@
 		(start 129.54 71.12)
 		(end 129.54 66.04)
-		(width 0.2)
+		(width 0.8)
 		(layer "B.Cu")
 		(net 1)
@@
 		(start 142.24 88.9)
 		(end 157.48 88.9)
-		(width 0.2)
+		(width 0.8)
 		(layer "B.Cu")
 		(net 1)
@@
 		(start 132.08 88.9)
 		(end 132.08 93.98)
-		(width 0.2)
+		(width 0.8)
 		(layer "B.Cu")
 		(net 1)
@@
 		(start 127 68.58)
 		(end 124.46 68.58)
-		(width 0.2)
+		(width 0.8)
 		(layer "F.Cu")
 		(net 2)
@@
 		(start 147.32 68.58)
 		(end 144.78 68.58)
-		(width 0.2)
+		(width 0.8)
 		(layer "B.Cu")
 		(net 2)
@@
 		(start 129.58 73.66)
 		(end 129.54 73.62)
-		(width 0.2)
+		(width 0.8)
 		(layer "B.Cu")
 		(net 2)
@@
 		(start 129.54 73.62)
 		(end 127.04 73.62)
-		(width 0.2)
+		(width 0.8)
 		(layer "B.Cu")
 		(net 2)
@@
 		(start 132.08 73.66)
 		(end 134.62 73.66)
-		(width 0.2)
+		(width 0.8)
 		(layer "B.Cu")
 		(net 2)
@@
 		(start 144.78 83.82)
 		(end 139.7 83.82)
-		(width 0.2)
+		(width 0.8)
 		(layer "B.Cu")
 		(net 2)
@@
 		(start 154.94 53.34)
 		(end 147.32 53.34)
-		(width 0.2)
+		(width 0.8)
 		(layer "B.Cu")
 		(net 2)
@@
 		(start 139.7 78.74)
 		(end 139.7 83.82)
-		(width 0.2)
+		(width 0.8)
 		(layer "B.Cu")
 		(net 2)
@@
 		(start 127 73.66)
 		(end 127 68.58)
-		(width 0.2)
+		(width 0.8)
 		(layer "B.Cu")
 		(net 2)
@@
 		(start 144.78 68.58)
 		(end 144.78 83.82)
-		(width 0.2)
+		(width 0.8)
 		(layer "B.Cu")
 		(net 2)
@@
 		(start 147.32 53.34)
 		(end 147.32 68.58)
-		(width 0.2)
+		(width 0.8)
 		(layer "B.Cu")
 		(net 2)
@@
 		(start 127.04 73.62)
 		(end 127 73.66)
-		(width 0.2)
+		(width 0.8)
 		(layer "B.Cu")
 		(net 2)
@@
 		(start 132.08 73.66)
 		(end 129.58 73.66)
-		(width 0.2)
+		(width 0.8)
 		(layer "B.Cu")
 		(net 2)
@@
 		(start 139.7 78.74)
 		(end 134.62 78.74)
-		(width 0.2)
+		(width 0.8)
 		(layer "B.Cu")
 		(net 2)
@@
 		(start 134.62 73.66)
 		(end 134.62 78.74)
-		(width 0.2)
+		(width 0.8)
 		(layer "B.Cu")
 		(net 2)
@@
 		(start 157.44 50.84)
 		(end 157.48 50.8)
-		(width 0.2)
+		(width 0.8)
 		(layer "B.Cu")
 		(net 3)
@@
 		(start 142.24 53.34)
 		(end 142.24 50.8)
-		(width 0.2)
+		(width 0.8)
 		(layer "B.Cu")
 		(net 3)
@@
 		(start 142.24 50.8)
 		(end 147.32 50.8)
-		(width 0.2)
+		(width 0.8)
 		(layer "B.Cu")
 		(net 3)
@@
 		(start 154.9 50.8)
 		(end 154.94 50.84)
-		(width 0.2)
+		(width 0.8)
 		(layer "B.Cu")
 		(net 3)
@@
 		(start 147.32 50.8)
 		(end 154.9 50.8)
-		(width 0.2)
+		(width 0.8)
 		(layer "B.Cu")
 		(net 3)
@@
 		(start 139.7 53.34)
 		(end 142.24 53.34)
-		(width 0.2)
+		(width 0.8)
 		(layer "B.Cu")
 		(net 3)
@@
 		(start 154.94 50.84)
 		(end 157.44 50.84)
-		(width 0.2)
+		(width 0.8)
 		(layer "B.Cu")
 		(net 3)
@@
 		(start 157.48 58.42)
 		(end 157.48 60.96)
-		(width 0.2)
+		(width 0.8)
 		(layer "B.Cu")
 		(net 3)
@@
 		(start 157.48 50.8)
 		(end 157.48 58.42)
-		(width 0.2)
+		(width 0.8)
 		(layer "B.Cu")
 		(net 3)
@@
 		(start 142.24 106.68)
 		(end 127 106.68)
-		(width 0.2)
+		(width 0.8)
 		(layer "B.Cu")
 		(net 7)
@@
 		(start 142.24 109.22)
 		(end 142.24 106.68)
-		(width 0.2)
+		(width 0.8)
 		(layer "B.Cu")
 		(net 7)
@@
 		(start 127 78.74)
 		(end 132.08 78.74)
-		(width 0.2)
+		(width 0.8)
 		(layer "B.Cu")
 		(net 7)
@@
 		(start 127 106.68)
 		(end 127 78.74)
-		(width 0.2)
+		(width 0.8)
 		(layer "B.Cu")
 		(net 7)
@@
 		(start 129.54 104.14)
 		(end 144.78 104.14)
-		(width 0.2)
+		(width 0.8)
 		(layer "B.Cu")
 		(net 8)
@@
 		(start 132.08 81.28)
 		(end 129.54 81.28)
-		(width 0.2)
+		(width 0.8)
 		(layer "B.Cu")
 		(net 8)
@@
 		(start 144.78 104.14)
 		(end 144.78 109.22)
-		(width 0.2)
+		(width 0.8)
 		(layer "B.Cu")
 		(net 8)
@@
 		(start 129.54 81.28)
 		(end 129.54 104.14)
-		(width 0.2)
+		(width 0.8)
 		(layer "B.Cu")
 		(net 8)
@@
 		(start 142.24 76.2)
 		(end 142.24 81.28)
-		(width 0.2)
+		(width 0.8)
 		(layer "B.Cu")
 		(net 20)
@@
 		(start 139.7 76.2)
 		(end 142.24 76.2)
-		(width 0.2)
+		(width 0.8)
 		(layer "B.Cu")
 		(net 20)
@@
 		(start 152.4 63.5)
 		(end 157.48 63.5)
-		(width 0.2)
+		(width 0.8)
 		(layer "B.Cu")
 		(net 39)
@@
 		(start 157.48 63.5)
 		(end 157.48 66.12)
-		(width 0.2)
+		(width 0.8)
 		(layer "B.Cu")
 		(net 39)
@@
 		(start 152.4 66.04)
 		(end 154.94 66.04)
-		(width 0.2)
+		(width 0.8)
 		(layer "B.Cu")
 		(net 40)
@@
 		(start 154.94 68.58)
 		(end 157.44 68.58)
-		(width 0.2)
+		(width 0.8)
 		(layer "B.Cu")
 		(net 40)
@@
 		(start 157.44 68.58)
 		(end 157.48 68.62)
-		(width 0.2)
+		(width 0.8)
 		(layer "B.Cu")
 		(net 40)
@@
 		(start 154.94 66.04)
 		(end 154.94 68.58)
-		(width 0.2)
+		(width 0.8)
 		(layer "B.Cu")
 		(net 40)
@@
 		(start 144.78 55.88)
 		(end 144.78 63.5)
-		(width 0.2)
+		(width 0.8)
 		(layer "B.Cu")
 		(net 45)
@@
 		(start 139.7 55.88)
 		(end 144.78 55.88)
-		(width 0.2)
+		(width 0.8)
 		(layer "B.Cu")
 		(net 45)
@@
 		(start 139.7 58.42)
 		(end 142.24 58.42)
-		(width 0.2)
+		(width 0.8)
 		(layer "B.Cu")
 		(net 46)
@@
 		(start 142.24 58.42)
 		(end 142.24 66.04)
-		(width 0.2)
+		(width 0.8)
 		(layer "B.Cu")
 		(net 46)
@@
 		(start 142.24 66.04)
 		(end 144.78 66.04)
-		(width 0.2)
+		(width 0.8)
 		(layer "B.Cu")
 		(net 46)
